File: Beta/PistormX 1K2 alt/KiCAD/PistormX1K2.kicad_sch (KiCad schematic)
At the start: 30 parts, among them CN1 FCN-225J150-GA_90deg_A1200, J1 EXT, J2 Raspberry_Pi_2_3, J3 PROG, J4 EXT2, U1 XC95288XL-TQ144, U2 SPX3819M5-L-3-3, U3 XC6206PxxxMR, U9 AMS1117-3.3

Commit message: Added an alternative board layout for the Pistorm'X 1K2. Some cleanup on the first PiStorm'X 1K2 board. Updated README.
Parts:
- J2: footprint Sassa:PinSocket_2x20_P2.54mm_Vertical_SMD_BottomEntry -> Sassa:PinSocket_2x20_P2.54mm_Vertical_SMD+THT_DoubleSide
Connections:
- net A0: now also U1.40 (P40); no longer U1.116 (P116)
- net A1: now also U1.45 (P45); no longer U1.115 (P115)
- net A10: now also U1.53 (P53); no longer U1.88 (P88)
- net A11: now also U1.56 (P56); no longer U1.87 (P87)
- net A12: now also U1.54 (P54); no longer U1.83 (P83)
- net A13: now also U1.57 (P57); no longer U1.82 (P82)
- net A14: now also U1.58 (P58); no longer U1.79 (P79)
- net A15: now also U1.60 (P60); no longer U1.78 (P78)
- net A16: now also U1.59 (P59); no longer U1.76 (P76)
- net A17: now also U1.66 (P66); no longer U1.70 (P70)
- net A18: now also U1.61 (P61); no longer U1.66 (P66)
- net A19: now also U1.68 (P68); no longer U1.57 (P57)
- net A2: now also U1.43 (P43); no longer U1.113 (P113)
- net A20: now also U1.64 (P64); no longer U1.56 (P56)
- net A21: now also U1.70 (P70); no longer U1.53 (P53)
- net A22: now also U1.69 (P69); no longer U1.52 (P52)
- net A23: now also U1.71 (P71); no longer U1.51 (P51)
- net A3: now also U1.44 (P44); no longer U1.112 (P112)
- net A4: now also U1.46 (P46); no longer U1.96 (P96)
- net A5: now also U1.49 (P49); no longer U1.110 (P110)
- net A6: now also U1.48 (P48); no longer U1.111 (P111)
- net A7: now also U1.50 (P50); no longer U1.95 (P95)
- net A8: now also U1.51 (P51); no longer U1.93 (P93)
- net A9: now also U1.52 (P52); no longer U1.92 (P92)
- net D0: now also U1.21 (P21); no longer U1.11 (P11)
- net D1: now also U1.20 (P20); no longer U1.133 (P133)
- net D10: now also U1.142 (P142); no longer U1.2 (I/O/GTS3)
- net D11: now also U1.140 (P140); no longer U1.131 (P131)
- net D12: now also U1.139 (P139); no longer U1.142 (P142)
- net D13: now also U1.138 (P138); no longer U1.143 (I/O/GSR)
- net D14: now also U1.137 (P137); no longer U1.140 (P140)
- net D15: now also U1.136 (P136); no longer U1.130 (P130)
- net D16: now also U1.134 (P134); no longer U1.139 (P139)
- net D17: now also U1.131 (P131); no longer U1.129 (P129)
- net D18: now also U1.133 (P133); no longer U1.137 (P137)
- net D19: now also U1.130 (P130); no longer U1.138 (P138)
- net D2: now also U1.24 (P24); no longer U1.10 (P10)
- net D20: now also U1.128 (P128); no longer U1.136 (P136)
- net D21: now also U1.124 (P124); no longer U1.128 (P128)
- net D22: now also U1.117 (P117); no longer U1.134 (P134)
- net D23: now also U1.119 (P119); no longer U1.135 (P135)
- net D24: now also U1.116 (P116); no longer U1.126 (P126)
- net D25: now also U1.112 (P112); no longer U1.125 (P125)
- net D26: now also U1.115 (P115); no longer U1.124 (P124)
- net D27: now also U1.111 (P111); no longer U1.121 (P121)
- net D28: now also U1.38 (I/O/GCK3); no longer U1.120 (P120)
- net D29: now also U1.113 (P113); no longer U1.119 (P119)
- net D3: now also U1.17 (P17); no longer U1.9 (P9)
- net D30: now also U1.39 (P39); no longer U1.118 (P118)
- net D31: now also U1.41 (P41); no longer U1.117 (P117)
- net D4: now also U1.15 (P15); no longer U1.7 (P7)
- net D5: now also U1.13 (P13); no longer U1.132 (P132)
- net D6: now also U1.11 (P11); no longer U1.6 (I/O/GTS2)
- net D7: now also U1.6 (I/O/GTS2); no longer U1.5 (I/O/GTS1)
- net D8: now also U1.3 (I/O/GTS4); no longer U1.4 (P4)
- net D9: now also U1.143 (I/O/GSR); no longer U1.3 (I/O/GTS4)
- net FC0: now also U1.5 (I/O/GTS1); no longer U1.27 (P27)
- net FC1: now also U1.25 (P25); no longer U1.26 (P26)
- net GPIO0: now also U1.103 (P103); no longer U1.74 (P74)
- net GPIO1: now also U1.102 (P102); no longer U1.75 (P75)
- net GPIO10: now also U1.77 (P77); no longer U1.91 (P91)
- net GPIO11: now also U1.105 (P105); no longer U1.80 (P80)
- net GPIO12: now also U1.98 (P98); no longer U1.69 (P69)
- net GPIO13: now also U1.96 (P96); no longer U1.64 (P64)
- net GPIO14: now also U1.91 (P91); no longer U1.104 (P104)
- net GPIO15: now also U1.85 (P85); no longer U1.103 (P103)
- net GPIO16: now also U1.94 (P94); no longer U1.60 (P60)
- net GPIO17: now also U1.83 (P83); no longer U1.102 (P102)
- net GPIO18: now also U1.82 (P82); no longer U1.101 (P101)
- net GPIO19: now also U1.92 (P92); no longer U1.59 (P59)
- net GPIO2: now also U1.97 (P97); no longer U1.107 (P107)
- net GPIO20: now also U1.86 (P86); no longer U1.61 (P61)
- net GPIO21: now also U1.87 (P87); no longer U1.54 (P54)
- net GPIO22: now also U1.80 (P80); no longer U1.97 (P97)
- net GPIO23: now also U1.79 (P79); no longer U1.98 (P98)
- net GPIO24: now also U1.78 (P78); no longer U1.94 (P94)
- net GPIO25: now also U1.75 (P75); no longer U1.86 (P86)
- net GPIO26: now also U1.88 (P88); no longer U1.58 (P58)
- net GPIO27: now also U1.81 (P81); no longer U1.100 (P100)
- net GPIO3: now also U1.95 (P95); no longer U1.106 (P106)
- net GPIO4: now also U1.93 (P93); no longer U1.105 (P105)
- net GPIO5: now also U1.101 (P101); no longer U1.71 (P71)
- net GPIO6: now also U1.100 (P100); no longer U1.68 (P68)
- net GPIO7: now also U1.104 (P104); no longer U1.77 (P77)
- net GPIO8: now also U1.74 (P74); no longer U1.81 (P81)
- net GPIO9: now also U1.76 (P76); no longer U1.85 (P85)
- net RW: now also U1.12 (P12); no longer U1.22 (P22)
- net SIZ0: now also U1.32 (I/O/GCK2); no longer U1.17 (P17)
- net SIZ1: now also U1.14 (P14); no longer U1.19 (P19)
- net SPARE0: now also U1.120 (P120); no longer U1.38 (I/O/GCK3)
- net SPARE1: now also U1.118 (P118); no longer U1.39 (P39)
- net SPARE2: now also U1.125 (P125); no longer U1.40 (P40)
- net SPARE3: now also U1.121 (P121); no longer U1.41 (P41)
- net SPARE4: now also U1.129 (P129); no longer U1.43 (P43)
- net SPARE5: now also U1.126 (P126); no longer U1.44 (P44)
- net SPARE6: now also U1.135 (P135); no longer U1.45 (P45)
- net SPARE7: now also U1.132 (P132); no longer U1.46 (P46)
- net SPAREA: now also U1.106 (P106); no longer U1.48 (P48)
- net SPAREB: now also U1.107 (P107); no longer U1.49 (P49)
- net SPAREC: now also U1.110 (P110); no longer U1.50 (P50)
- net TCK: now also J3.3 (Pin_3); no longer J3.4 (Pin_4)
- net TDI: now also J3.5 (Pin_5); no longer J3.6 (Pin_6)
- net TDO: now also J3.6 (Pin_6); no longer J3.3 (Pin_3)
- net TMS: now also J3.4 (Pin_4); no longer J3.5 (Pin_5)
- net _AS: now also U1.31 (P31); no longer U1.20 (P20)
- net _BERR: now also U1.27 (P27); no longer U1.23 (P23)
- net _BG: now also U1.22 (P22); no longer U1.28 (P28)
- net _BR: now also U1.23 (P23); no longer U1.31 (P31)
- net _DS: now also U1.28 (P28); no longer U1.21 (P21)
- net _DSACK0: now also U1.26 (P26); no longer U1.24 (P24)
- net _DSACK1: now also U1.9 (P9); no longer U1.25 (P25)
- net _HALT: now also U1.33 (P33); no longer U1.16 (P16)
- net _INT2: now also U1.2 (I/O/GTS3); no longer U1.35 (P35)
- net _INT6: now also U1.4 (P4); no longer U1.34 (P34)
- net _IPL0: now also U1.35 (P35); no longer U1.14 (P14)
- net _IPL1: now also U1.34 (P34); no longer U1.13 (P13)
- net _IPL2: now also U1.19 (P19); no longer U1.12 (P12)
- net _KB_RESET: now also U1.10 (P10); no longer U1.32 (I/O/GCK2)
- net _OVR: now also U1.7 (P7); no longer U1.33 (P33)
- net _RST: now also U1.16 (P16); no longer U1.15 (P15)
