File: Beta/PistormX 500 DIP/KiCAD/PistormX500.kicad_pcb (KiCad board)
At the start: 2 copper layers, 82.6 x 34.3 mm, 25 parts, among them J1 68000D socket, J2 Raspberry_Pi_2_3, J3 PROG, J4 OVR, U1 XC95144XL-TQ100, U2 SPX3819M5-L-3-3, U3 XC6206PxxxMR, U4 CY62177ESL-55ZXI

Commit message: PiStorm'X 500 and PiStorm'X 600 corrections. PiStorm'X 600 is actually working and under test. PiStorm'X 500 will be tested after I find an Agnus 8375 or A500 motherboard replacement.
Other:
- rule pad_to_mask_clearance: 0 -> 0.038
Changed lines of the file:
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@@
       (dielectric_constraints no)
     )
-    (pad_to_mask_clearance 0)
+    (pad_to_mask_clearance 0.038)
+    (solder_mask_min_width 0.1)
     (pcbplotparams
       (layerselection 0x00010fc_ffffffff)
